File: electronics/q5/mcu-5.kicad_sch (KiCad schematic)
At the start: 6 parts, among them SW2 RESET COUNT / BOOT, SW3 MCU RESET

Commit message: WIP: Q5 design-lock routing iteration snapshot (not verified)
Co-Authored-By: Claude Opus 5.5 <noreply@anthropic.com>
Claude-Session: https://claude.ai/code/session_01UrkzLMrBi6iLPSL5SbMCA7
Parts:
- SW2: footprint CountFidgetQ5:HanElectricity_CPG151101D13_MX_Plate -> CountFidgetQ5:SW_Hotswap_Kailh_MX_CPG151101S11; MPN CPG151101D13 -> CPG151101S11-16
Changed lines of the file:
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@@
       (in_bom yes) (on_board yes) (dnp no)
  (property "Reference" "SW2" (at 105.41 73.66 0) (effects (font (size 1.524 1.524)))) (property "Value" "RESET COUNT / BOOT" (at 105.41 77.46999999999998 0) (effects (font (size 1.524 1.524))))
-      (property "Footprint" "CountFidgetQ5:HanElectricity_CPG151101D13_MX_Plate" (at 105.41 82.55 0) (effects (font (size 1.27 1.27)) (hide yes))) (property "MPN" "CPG151101D13" (at 105.41 77.46999999999998 0) (effects (font (size 1.524 1.524)) (hide yes)))
-      (property "Description" "Exact clicky switch; home through-hole soldering after rear key plate is fitted. Verify body/plate/lead fit before soldering; vendor SMT assembly excludes this part." (at 105.41 82.55 0) (effects (font (size 1.27 1.27)) (hide yes)))
+      (property "Footprint" "CountFidgetQ5:SW_Hotswap_Kailh_MX_CPG151101S11" (at 105.41 82.55 0) (effects (font (size 1.27 1.27)) (hide yes))) (property "MPN" "CPG151101S11-16" (at 105.41 77.46999999999998 0) (effects (font (size 1.524 1.524)) (hide yes)))
+      (property "Description" "MX hot-swap socket, vendor SMT on the bottom side. RESET COUNT / BOOT0. The user presses a clicky MX switch (CPG151101D13, clipped into the printed key plate) into it: no switch soldering." (at 105.41 82.55 0) (effects (font (size 1.27 1.27)) (hide yes)))
       (pin "1")(pin "2")
       (instances (project "click-counter-Q5" (path "/7c190cd8-3ca2-5363-8a92-396d30a08243/2f9dfd4f-ef26-5940-ad4a-519e367606ec" (reference "SW2") (unit 1)))))
