File: electronics/q5/display-1.kicad_sch (KiCad schematic)
At the start: 6 parts

Commit message: Q5 design lock: JLC Basic substitutions, re-verified board, cost estimator
Co-Authored-By: Claude Opus 5.5 <noreply@anthropic.com>
Claude-Session: https://claude.ai/code/session_01UrkzLMrBi6iLPSL5SbMCA7
Parts:
- C20: MPN GRM188R71H104KA93D -> CC0603KRX7R9BB104
- C28: MPN GRM1885C1H472JA01D -> 0603B472K500NT
- R24, R25, R29: MPN RC0603FR-07100KL -> 0603WAF1003T5E
Changed lines of the file:
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@@
       (in_bom yes) (on_board yes) (dnp no)
  (property "Reference" "C20" (at 105.41 73.66 0) (effects (font (size 1.524 1.524)))) (property "Value" "100n" (at 105.41 77.46999999999998 0) (effects (font (size 1.524 1.524))))
-      (property "Footprint" "CountFidgetQ5:Capacitor_SMD_C_0603_1608Metric" (at 105.41 82.55 0) (effects (font (size 1.27 1.27)) (hide yes))) (property "MPN" "GRM188R71H104KA93D" (at 105.41 77.46999999999998 0) (effects (font (size 1.524 1.524)) (hide yes)))
+      (property "Footprint" "CountFidgetQ5:Capacitor_SMD_C_0603_1608Metric" (at 105.41 82.55 0) (effects (font (size 1.27 1.27)) (hide yes))) (property "MPN" "CC0603KRX7R9BB104" (at 105.41 77.46999999999998 0) (effects (font (size 1.524 1.524)) (hide yes)))
       (property "Description" "50V X7R +/-10%; at DS1.VDD." (at 105.41 82.55 0) (effects (font (size 1.27 1.27)) (hide yes)))
       (pin "1")(pin "2")
@@
       (in_bom yes) (on_board yes) (dnp no)
  (property "Reference" "C28" (at 294.64 73.66 0) (effects (font (size 1.524 1.524)))) (property "Value" "4.7n" (at 294.64 77.46999999999998 0) (effects (font (size 1.524 1.524))))
-      (property "Footprint" "CountFidgetQ5:Capacitor_SMD_C_0603_1608Metric" (at 294.64 82.55 0) (effects (font (size 1.27 1.27)) (hide yes))) (property "MPN" "GRM1885C1H472JA01D" (at 294.64 77.46999999999998 0) (effects (font (size 1.524 1.524)) (hide yes)))
-      (property "Description" "4.7nF 50V C0G slew capacitor to VIN; tON 17.9ms typical; typical slew only" (at 294.64 82.55 0) (effects (font (size 1.27 1.27)) (hide yes)))
+      (property "Footprint" "CountFidgetQ5:Capacitor_SMD_C_0603_1608Metric" (at 294.64 82.55 0) (effects (font (size 1.27 1.27)) (hide yes))) (property "MPN" "0603B472K500NT" (at 294.64 77.46999999999998 0) (effects (font (size 1.524 1.524)) (hide yes)))
+      (property "Description" "4.7nF 50V X7R slew capacitor to VIN; tON 17.9ms typical; typical slew only" (at 294.64 82.55 0) (effects (font (size 1.27 1.27)) (hide yes)))
       (pin "1")(pin "2")
       (instances (project "click-counter-Q5" (path "/7c190cd8-3ca2-5363-8a92-396d30a08243/a5c2d3a6-51db-5a84-b99b-2f2e9ec90a3a" (reference "C28") (unit 1)))))
@@
       (in_bom yes) (on_board yes) (dnp no)
  (property "Reference" "R24" (at 294.64 152.4 0) (effects (font (size 1.524 1.524)))) (property "Value" "100k" (at 294.64 156.21 0) (effects (font (size 1.524 1.524))))
-      (property "Footprint" "CountFidgetQ5:Resistor_SMD_R_0603_1608Metric" (at 294.64 161.29 0) (effects (font (size 1.27 1.27)) (hide yes))) (property "MPN" "RC0603FR-07100KL" (at 294.64 156.21 0) (effects (font (size 1.524 1.524)) (hide yes)))
+      (property "Footprint" "CountFidgetQ5:Resistor_SMD_R_0603_1608Metric" (at 294.64 161.29 0) (effects (font (size 1.27 1.27)) (hide yes))) (property "MPN" "0603WAF1003T5E" (at 294.64 156.21 0) (effects (font (size 1.524 1.524)) (hide yes)))
       (property "Description" "1%,100mW" (at 294.64 161.29 0) (effects (font (size 1.27 1.27)) (hide yes)))
       (pin "1")(pin "2")
@@
       (in_bom yes) (on_board yes) (dnp no)
  (property "Reference" "R25" (at 105.41 229.87 0) (effects (font (size 1.524 1.524)))) (property "Value" "100k" (at 105.41 233.68 0) (effects (font (size 1.524 1.524))))
-      (property "Footprint" "CountFidgetQ5:Resistor_SMD_R_0603_1608Metric" (at 105.41 238.76 0) (effects (font (size 1.27 1.27)) (hide yes))) (property "MPN" "RC0603FR-07100KL" (at 105.41 233.68 0) (effects (font (size 1.524 1.524)) (hide yes)))
+      (property "Footprint" "CountFidgetQ5:Resistor_SMD_R_0603_1608Metric" (at 105.41 238.76 0) (effects (font (size 1.27 1.27)) (hide yes))) (property "MPN" "0603WAF1003T5E" (at 105.41 233.68 0) (effects (font (size 1.524 1.524)) (hide yes)))
       (property "Description" "1%,100mW" (at 105.41 238.76 0) (effects (font (size 1.27 1.27)) (hide yes)))
       (pin "1")(pin "2")
@@
       (in_bom yes) (on_board yes) (dnp no)
  (property "Reference" "R29" (at 294.64 229.87 0) (effects (font (size 1.524 1.524)))) (property "Value" "100k" (at 294.64 233.68 0) (effects (font (size 1.524 1.524))))
-      (property "Footprint" "CountFidgetQ5:Resistor_SMD_R_0603_1608Metric" (at 294.64 238.76 0) (effects (font (size 1.27 1.27)) (hide yes))) (property "MPN" "RC0603FR-07100KL" (at 294.64 233.68 0) (effects (font (size 1.524 1.524)) (hide yes)))
+      (property "Footprint" "CountFidgetQ5:Resistor_SMD_R_0603_1608Metric" (at 294.64 238.76 0) (effects (font (size 1.27 1.27)) (hide yes))) (property "MPN" "0603WAF1003T5E" (at 294.64 233.68 0) (effects (font (size 1.524 1.524)) (hide yes)))
       (property "Description" "100k CS pull-up to switched module supply; never to always-on rail" (at 294.64 238.76 0) (effects (font (size 1.27 1.27)) (hide yes)))
       (pin "1")(pin "2")
