File: electronics/q5/mcu-1.kicad_sch (KiCad schematic)
At the start: 5 parts, among them U1 STM32L072CBT6

Commit message: Q5 design lock: JLC Basic substitutions, re-verified board, cost estimator
Co-Authored-By: Claude Opus 5.5 <noreply@anthropic.com>
Claude-Session: https://claude.ai/code/session_01UrkzLMrBi6iLPSL5SbMCA7
Parts:
- C31, C32, C33, C34: MPN GRM188R71H104KA93D -> CC0603KRX7R9BB104
Changed lines of the file:
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@@
       (in_bom yes) (on_board yes) (dnp no)
  (property "Reference" "C31" (at 309.88 66.04 0) (effects (font (size 1.524 1.524)))) (property "Value" "100n" (at 309.88 69.85 0) (effects (font (size 1.524 1.524))))
-      (property "Footprint" "CountFidgetQ5:Capacitor_SMD_C_0603_1608Metric" (at 309.88 74.93 0) (effects (font (size 1.27 1.27)) (hide yes))) (property "MPN" "GRM188R71H104KA93D" (at 309.88 69.85 0) (effects (font (size 1.524 1.524)) (hide yes)))
+      (property "Footprint" "CountFidgetQ5:Capacitor_SMD_C_0603_1608Metric" (at 309.88 74.93 0) (effects (font (size 1.27 1.27)) (hide yes))) (property "MPN" "CC0603KRX7R9BB104" (at 309.88 69.85 0) (effects (font (size 1.524 1.524)) (hide yes)))
       (property "Description" "100nF local STM32 supply bypass; one per VDD/VDDA/USB supply group" (at 309.88 74.93 0) (effects (font (size 1.27 1.27)) (hide yes)))
       (pin "1")(pin "2")
@@
       (in_bom yes) (on_board yes) (dnp no)
  (property "Reference" "C32" (at 309.88 114.3 0) (effects (font (size 1.524 1.524)))) (property "Value" "100n" (at 309.88 118.10999999999999 0) (effects (font (size 1.524 1.524))))
-      (property "Footprint" "CountFidgetQ5:Capacitor_SMD_C_0603_1608Metric" (at 309.88 123.19 0) (effects (font (size 1.27 1.27)) (hide yes))) (property "MPN" "GRM188R71H104KA93D" (at 309.88 118.10999999999999 0) (effects (font (size 1.524 1.524)) (hide yes)))
+      (property "Footprint" "CountFidgetQ5:Capacitor_SMD_C_0603_1608Metric" (at 309.88 123.19 0) (effects (font (size 1.27 1.27)) (hide yes))) (property "MPN" "CC0603KRX7R9BB104" (at 309.88 118.10999999999999 0) (effects (font (size 1.524 1.524)) (hide yes)))
       (property "Description" "100nF local STM32 supply bypass; one per VDD/VDDA/USB supply group" (at 309.88 123.19 0) (effects (font (size 1.27 1.27)) (hide yes)))
       (pin "1")(pin "2")
@@
       (in_bom yes) (on_board yes) (dnp no)
  (property "Reference" "C33" (at 309.88 162.56 0) (effects (font (size 1.524 1.524)))) (property "Value" "100n" (at 309.88 166.37 0) (effects (font (size 1.524 1.524))))
-      (property "Footprint" "CountFidgetQ5:Capacitor_SMD_C_0603_1608Metric" (at 309.88 171.45 0) (effects (font (size 1.27 1.27)) (hide yes))) (property "MPN" "GRM188R71H104KA93D" (at 309.88 166.37 0) (effects (font (size 1.524 1.524)) (hide yes)))
+      (property "Footprint" "CountFidgetQ5:Capacitor_SMD_C_0603_1608Metric" (at 309.88 171.45 0) (effects (font (size 1.27 1.27)) (hide yes))) (property "MPN" "CC0603KRX7R9BB104" (at 309.88 166.37 0) (effects (font (size 1.524 1.524)) (hide yes)))
       (property "Description" "100nF local STM32 supply bypass; one per VDD/VDDA/USB supply group" (at 309.88 171.45 0) (effects (font (size 1.27 1.27)) (hide yes)))
       (pin "1")(pin "2")
@@
       (in_bom yes) (on_board yes) (dnp no)
  (property "Reference" "C34" (at 309.88 209.55 0) (effects (font (size 1.524 1.524)))) (property "Value" "100n" (at 309.88 213.36 0) (effects (font (size 1.524 1.524))))
-      (property "Footprint" "CountFidgetQ5:Capacitor_SMD_C_0603_1608Metric" (at 309.88 218.44 0) (effects (font (size 1.27 1.27)) (hide yes))) (property "MPN" "GRM188R71H104KA93D" (at 309.88 213.36 0) (effects (font (size 1.524 1.524)) (hide yes)))
+      (property "Footprint" "CountFidgetQ5:Capacitor_SMD_C_0603_1608Metric" (at 309.88 218.44 0) (effects (font (size 1.27 1.27)) (hide yes))) (property "MPN" "CC0603KRX7R9BB104" (at 309.88 213.36 0) (effects (font (size 1.524 1.524)) (hide yes)))
       (property "Description" "100nF local STM32 supply bypass; one per VDD/VDDA/USB supply group" (at 309.88 218.44 0) (effects (font (size 1.27 1.27)) (hide yes)))
       (pin "1")(pin "2")
