File: electronics/q5/mcu-3.kicad_sch (KiCad schematic)
At the start: 6 parts, among them Q5 COUNT key level shift

Commit message: Q5 design lock: JLC Basic substitutions, re-verified board, cost estimator
Co-Authored-By: Claude Opus 5.5 <noreply@anthropic.com>
Claude-Session: https://claude.ai/code/session_01UrkzLMrBi6iLPSL5SbMCA7
Parts:
- C7: MPN GRM188R71H104KA93D -> CC0603KRX7R9BB104
- Q5: MPN 2N7002,215 -> 2N7002
Changed lines of the file:
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@@
       (in_bom yes) (on_board yes) (dnp no)
  (property "Reference" "C7" (at 105.41 73.66 0) (effects (font (size 1.524 1.524)))) (property "Value" "100n" (at 105.41 77.46999999999998 0) (effects (font (size 1.524 1.524))))
-      (property "Footprint" "CountFidgetQ5:Capacitor_SMD_C_0603_1608Metric" (at 105.41 82.55 0) (effects (font (size 1.27 1.27)) (hide yes))) (property "MPN" "GRM188R71H104KA93D" (at 105.41 77.46999999999998 0) (effects (font (size 1.524 1.524)) (hide yes)))
+      (property "Footprint" "CountFidgetQ5:Capacitor_SMD_C_0603_1608Metric" (at 105.41 82.55 0) (effects (font (size 1.27 1.27)) (hide yes))) (property "MPN" "CC0603KRX7R9BB104" (at 105.41 77.46999999999998 0) (effects (font (size 1.524 1.524)) (hide yes)))
       (property "Description" "100 nF MCU decoupler beside U1 DVCC/DVSS; short via connections required" (at 105.41 82.55 0) (effects (font (size 1.27 1.27)) (hide yes)))
       (pin "1")(pin "2")
@@
       (in_bom yes) (on_board yes) (dnp no)
  (property "Reference" "Q5" (at 294.64 224.79 0) (effects (font (size 1.524 1.524)))) (property "Value" "COUNT key level shift" (at 294.64 228.6 0) (effects (font (size 1.524 1.524)) (hide yes)))
-      (property "Footprint" "CountFidgetQ5:Package_TO_SOT_SMD_SOT-23" (at 294.64 238.76 0) (effects (font (size 1.27 1.27)) (hide yes))) (property "MPN" "2N7002,215" (at 294.64 228.6 0) (effects (font (size 1.524 1.524))))
+      (property "Footprint" "CountFidgetQ5:Package_TO_SOT_SMD_SOT-23" (at 294.64 238.76 0) (effects (font (size 1.27 1.27)) (hide yes))) (property "MPN" "2N7002" (at 294.64 228.6 0) (effects (font (size 1.524 1.524))))
       (property "Description" "Mirrors the SYS-referenced COUNT key onto the unchanged active-low COUNT_N (R17/C11) input." (at 294.64 238.76 0) (effects (font (size 1.27 1.27)) (hide yes)))
       (pin "1")(pin "2")(pin "3")
