File: electronics/q5/mcu-4.kicad_sch (KiCad schematic)
At the start: 6 parts, among them SW1 COUNT / POWER

Commit message: WIP: Q5 design-lock routing iteration snapshot (not verified)
Co-Authored-By: Claude Opus 5.5 <noreply@anthropic.com>
Claude-Session: https://claude.ai/code/session_01UrkzLMrBi6iLPSL5SbMCA7
Parts:
- SW1: footprint CountFidgetQ5:HanElectricity_CPG151101D13_MX_Plate -> CountFidgetQ5:SW_Hotswap_Kailh_MX_CPG151101S11; MPN CPG151101D13 -> CPG151101S11-16
Changed lines of the file:
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@@
       (in_bom yes) (on_board yes) (dnp no)
  (property "Reference" "SW1" (at 294.64 229.87 0) (effects (font (size 1.524 1.524)))) (property "Value" "COUNT / POWER" (at 294.64 233.68 0) (effects (font (size 1.524 1.524))))
-      (property "Footprint" "CountFidgetQ5:HanElectricity_CPG151101D13_MX_Plate" (at 294.64 238.76 0) (effects (font (size 1.27 1.27)) (hide yes))) (property "MPN" "CPG151101D13" (at 294.64 233.68 0) (effects (font (size 1.524 1.524)) (hide yes)))
-      (property "Description" "Exact clicky switch closing SYS to PWR_KEY: powers the board on and, through Q5, drives COUNT_N low. Home through-hole soldering after the rear key plate is fitted." (at 294.64 238.76 0) (effects (font (size 1.27 1.27)) (hide yes)))
+      (property "Footprint" "CountFidgetQ5:SW_Hotswap_Kailh_MX_CPG151101S11" (at 294.64 238.76 0) (effects (font (size 1.27 1.27)) (hide yes))) (property "MPN" "CPG151101S11-16" (at 294.64 233.68 0) (effects (font (size 1.524 1.524)) (hide yes)))
+      (property "Description" "MX hot-swap socket, vendor SMT on the bottom side. COUNT / POWER: closes SYS to PWR_KEY, powering the board on and, through Q5, driving COUNT_N low. The user presses a clicky MX switch (CPG151101D13, clipped into the printed key plate) into it: no switch soldering." (at 294.64 238.76 0) (effects (font (size 1.27 1.27)) (hide yes)))
       (pin "1")(pin "2")
       (instances (project "click-counter-Q5" (path "/7c190cd8-3ca2-5363-8a92-396d30a08243/5b560024-5f43-580a-88a1-035a458454bd" (reference "SW1") (unit 1)))))

Commit message: Q5 design lock: JLC Basic substitutions, re-verified board, cost estimator
Co-Authored-By: Claude Opus 5.5 <noreply@anthropic.com>
Claude-Session: https://claude.ai/code/session_01UrkzLMrBi6iLPSL5SbMCA7
Parts:
- R16: MPN RC0603FR-0710KL -> 0603WAF1002T5E
- R18: MPN RC0603FR-07100KL -> 0603WAF1003T5E
Changed lines of the file:
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@@
       (in_bom yes) (on_board yes) (dnp no)
  (property "Reference" "R16" (at 105.41 73.66 0) (effects (font (size 1.524 1.524)))) (property "Value" "10k" (at 105.41 77.46999999999998 0) (effects (font (size 1.524 1.524))))
-      (property "Footprint" "CountFidgetQ5:Resistor_SMD_R_0603_1608Metric" (at 105.41 82.55 0) (effects (font (size 1.27 1.27)) (hide yes))) (property "MPN" "RC0603FR-0710KL" (at 105.41 77.46999999999998 0) (effects (font (size 1.524 1.524)) (hide yes)))
+      (property "Footprint" "CountFidgetQ5:Resistor_SMD_R_0603_1608Metric" (at 105.41 82.55 0) (effects (font (size 1.27 1.27)) (hide yes))) (property "MPN" "0603WAF1002T5E" (at 105.41 77.46999999999998 0) (effects (font (size 1.524 1.524)) (hide yes)))
       (property "Description" "1%, 0603, 0.1 W" (at 105.41 82.55 0) (effects (font (size 1.27 1.27)) (hide yes)))
       (pin "1")(pin "2")
@@
       (in_bom yes) (on_board yes) (dnp no)
  (property "Reference" "R18" (at 105.41 152.4 0) (effects (font (size 1.524 1.524)))) (property "Value" "100k" (at 105.41 156.21 0) (effects (font (size 1.524 1.524))))
-      (property "Footprint" "CountFidgetQ5:Resistor_SMD_R_0603_1608Metric" (at 105.41 161.29 0) (effects (font (size 1.27 1.27)) (hide yes))) (property "MPN" "RC0603FR-07100KL" (at 105.41 156.21 0) (effects (font (size 1.524 1.524)) (hide yes)))
+      (property "Footprint" "CountFidgetQ5:Resistor_SMD_R_0603_1608Metric" (at 105.41 161.29 0) (effects (font (size 1.27 1.27)) (hide yes))) (property "MPN" "0603WAF1003T5E" (at 105.41 156.21 0) (effects (font (size 1.524 1.524)) (hide yes)))
       (property "Description" "1%, 0603, 0.1 W; >=13.4 uA held-contact current at 2.97 V, above switch 10 uA minimum" (at 105.41 161.29 0) (effects (font (size 1.27 1.27)) (hide yes)))
       (pin "1")(pin "2")
