File: electronics/q5/usb-power-3.kicad_sch (KiCad schematic)
At the start: 6 parts, among them J1 USB-C power and DFU

Commit message: WIP: Q5 design-lock routing iteration snapshot (not verified)
Co-Authored-By: Claude Opus 5.5 <noreply@anthropic.com>
Claude-Session: https://claude.ai/code/session_01UrkzLMrBi6iLPSL5SbMCA7
Parts:
- removed R30: 150k, CountFidgetQ5:Resistor_SMD_R_0603_1608Metric, symbol CountFidgetQ5:R30
- added D4: 1N4148WS, CountFidgetQ5:Diode_SMD_D_SOD-323, symbol CountFidgetQ5:D4
Connections:
- net VBUS: now also D4.2 (A)
- new net VBUS_WAKE: D4.1 (K)
Other:
- moved on the sheet: J1, R1, R19, R2, R3

Commit message: Q5 design lock: JLC Basic substitutions, re-verified board, cost estimator
Co-Authored-By: Claude Opus 5.5 <noreply@anthropic.com>
Claude-Session: https://claude.ai/code/session_01UrkzLMrBi6iLPSL5SbMCA7
Parts:
- R1, R2: MPN RC0603FR-075K1L -> 0603WAF5101T5E
- R19: MPN RC0603FR-072KL -> 0603WAF2001T5E
Changed lines of the file:
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@@
       (in_bom yes) (on_board yes) (dnp no)
  (property "Reference" "R1" (at 105.41 152.4 0) (effects (font (size 1.524 1.524)))) (property "Value" "5.1k" (at 105.41 156.21 0) (effects (font (size 1.524 1.524))))
-      (property "Footprint" "CountFidgetQ5:Resistor_SMD_R_0603_1608Metric" (at 105.41 161.29 0) (effects (font (size 1.27 1.27)) (hide yes))) (property "MPN" "RC0603FR-075K1L" (at 105.41 156.21 0) (effects (font (size 1.524 1.524)) (hide yes)))
+      (property "Footprint" "CountFidgetQ5:Resistor_SMD_R_0603_1608Metric" (at 105.41 161.29 0) (effects (font (size 1.27 1.27)) (hide yes))) (property "MPN" "0603WAF5101T5E" (at 105.41 156.21 0) (effects (font (size 1.524 1.524)) (hide yes)))
       (property "Description" "1%, 0603, 0.1 W" (at 105.41 161.29 0) (effects (font (size 1.27 1.27)) (hide yes)))
       (pin "1")(pin "2")
@@
       (in_bom yes) (on_board yes) (dnp no)
  (property "Reference" "R19" (at 294.64 152.4 0) (effects (font (size 1.524 1.524)))) (property "Value" "2k" (at 294.64 156.21 0) (effects (font (size 1.524 1.524))))
-      (property "Footprint" "CountFidgetQ5:Resistor_SMD_R_0603_1608Metric" (at 294.64 161.29 0) (effects (font (size 1.27 1.27)) (hide yes))) (property "MPN" "RC0603FR-072KL" (at 294.64 156.21 0) (effects (font (size 1.524 1.524)) (hide yes)))
+      (property "Footprint" "CountFidgetQ5:Resistor_SMD_R_0603_1608Metric" (at 294.64 161.29 0) (effects (font (size 1.27 1.27)) (hide yes))) (property "MPN" "0603WAF2001T5E" (at 294.64 156.21 0) (effects (font (size 1.524 1.524)) (hide yes)))
       (property "Description" "1%, 0603, 0.1 W" (at 294.64 161.29 0) (effects (font (size 1.27 1.27)) (hide yes)))
       (pin "1")(pin "2")
@@
       (in_bom yes) (on_board yes) (dnp no)
  (property "Reference" "R2" (at 105.41 229.87 0) (effects (font (size 1.524 1.524)))) (property "Value" "5.1k" (at 105.41 233.68 0) (effects (font (size 1.524 1.524))))
-      (property "Footprint" "CountFidgetQ5:Resistor_SMD_R_0603_1608Metric" (at 105.41 238.76 0) (effects (font (size 1.27 1.27)) (hide yes))) (property "MPN" "RC0603FR-075K1L" (at 105.41 233.68 0) (effects (font (size 1.524 1.524)) (hide yes)))
+      (property "Footprint" "CountFidgetQ5:Resistor_SMD_R_0603_1608Metric" (at 105.41 238.76 0) (effects (font (size 1.27 1.27)) (hide yes))) (property "MPN" "0603WAF5101T5E" (at 105.41 233.68 0) (effects (font (size 1.524 1.524)) (hide yes)))
       (property "Description" "1%, 0603, 0.1 W" (at 105.41 238.76 0) (effects (font (size 1.27 1.27)) (hide yes)))
       (pin "1")(pin "2")
