File: electronics/q5/mcu-2.kicad_sch (KiCad schematic)
At the start: 6 parts

Commit message: Q5 design lock: JLC Basic substitutions, re-verified board, cost estimator
Co-Authored-By: Claude Opus 5.5 <noreply@anthropic.com>
Claude-Session: https://claude.ai/code/session_01UrkzLMrBi6iLPSL5SbMCA7
Parts:
- C10, C35, C37: MPN GRM188R71H104KA93D -> CC0603KRX7R9BB104
- C11, C12: MPN GRM1885C1H102JA01D -> CL10B102KB8NNNC
Changed lines of the file:
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@@
       (in_bom yes) (on_board yes) (dnp no)
  (property "Reference" "C10" (at 105.41 73.66 0) (effects (font (size 1.524 1.524)))) (property "Value" "100n" (at 105.41 77.46999999999998 0) (effects (font (size 1.524 1.524))))
-      (property "Footprint" "CountFidgetQ5:Capacitor_SMD_C_0603_1608Metric" (at 105.41 82.55 0) (effects (font (size 1.27 1.27)) (hide yes))) (property "MPN" "GRM188R71H104KA93D" (at 105.41 77.46999999999998 0) (effects (font (size 1.524 1.524)) (hide yes)))
+      (property "Footprint" "CountFidgetQ5:Capacitor_SMD_C_0603_1608Metric" (at 105.41 82.55 0) (effects (font (size 1.27 1.27)) (hide yes))) (property "MPN" "CC0603KRX7R9BB104" (at 105.41 77.46999999999998 0) (effects (font (size 1.524 1.524)) (hide yes)))
       (property "Description" "100nF NRST bypass; recovery switch/test pad access required" (at 105.41 82.55 0) (effects (font (size 1.27 1.27)) (hide yes)))
       (pin "1")(pin "2")
@@
       (in_bom yes) (on_board yes) (dnp no)
  (property "Reference" "C11" (at 294.64 73.66 0) (effects (font (size 1.524 1.524)))) (property "Value" "1n" (at 294.64 77.46999999999998 0) (effects (font (size 1.524 1.524))))
-      (property "Footprint" "CountFidgetQ5:Capacitor_SMD_C_0603_1608Metric" (at 294.64 82.55 0) (effects (font (size 1.27 1.27)) (hide yes))) (property "MPN" "GRM1885C1H102JA01D" (at 294.64 77.46999999999998 0) (effects (font (size 1.524 1.524)) (hide yes)))
-      (property "Description" "1 nF, 50 V, C0G" (at 294.64 82.55 0) (effects (font (size 1.27 1.27)) (hide yes)))
+      (property "Footprint" "CountFidgetQ5:Capacitor_SMD_C_0603_1608Metric" (at 294.64 82.55 0) (effects (font (size 1.27 1.27)) (hide yes))) (property "MPN" "CL10B102KB8NNNC" (at 294.64 77.46999999999998 0) (effects (font (size 1.524 1.524)) (hide yes)))
+      (property "Description" "1 nF, 50 V, X7R" (at 294.64 82.55 0) (effects (font (size 1.27 1.27)) (hide yes)))
       (pin "1")(pin "2")
       (instances (project "click-counter-Q5" (path "/7c190cd8-3ca2-5363-8a92-396d30a08243/25c8a497-d064-5849-8b98-8381803a397d" (reference "C11") (unit 1)))))
@@
       (in_bom yes) (on_board yes) (dnp no)
  (property "Reference" "C12" (at 105.41 152.4 0) (effects (font (size 1.524 1.524)))) (property "Value" "1n" (at 105.41 156.21 0) (effects (font (size 1.524 1.524))))
-      (property "Footprint" "CountFidgetQ5:Capacitor_SMD_C_0603_1608Metric" (at 105.41 161.29 0) (effects (font (size 1.27 1.27)) (hide yes))) (property "MPN" "GRM1885C1H102JA01D" (at 105.41 156.21 0) (effects (font (size 1.524 1.524)) (hide yes)))
-      (property "Description" "1 nF, 50 V, C0G" (at 105.41 161.29 0) (effects (font (size 1.27 1.27)) (hide yes)))
+      (property "Footprint" "CountFidgetQ5:Capacitor_SMD_C_0603_1608Metric" (at 105.41 161.29 0) (effects (font (size 1.27 1.27)) (hide yes))) (property "MPN" "CL10B102KB8NNNC" (at 105.41 156.21 0) (effects (font (size 1.524 1.524)) (hide yes)))
+      (property "Description" "1 nF, 50 V, X7R" (at 105.41 161.29 0) (effects (font (size 1.27 1.27)) (hide yes)))
       (pin "1")(pin "2")
       (instances (project "click-counter-Q5" (path "/7c190cd8-3ca2-5363-8a92-396d30a08243/25c8a497-d064-5849-8b98-8381803a397d" (reference "C12") (unit 1)))))
@@
       (in_bom yes) (on_board yes) (dnp no)
  (property "Reference" "C35" (at 294.64 152.4 0) (effects (font (size 1.524 1.524)))) (property "Value" "100n" (at 294.64 156.21 0) (effects (font (size 1.524 1.524))))
-      (property "Footprint" "CountFidgetQ5:Capacitor_SMD_C_0603_1608Metric" (at 294.64 161.29 0) (effects (font (size 1.27 1.27)) (hide yes))) (property "MPN" "GRM188R71H104KA93D" (at 294.64 156.21 0) (effects (font (size 1.524 1.524)) (hide yes)))
+      (property "Footprint" "CountFidgetQ5:Capacitor_SMD_C_0603_1608Metric" (at 294.64 161.29 0) (effects (font (size 1.27 1.27)) (hide yes))) (property "MPN" "CC0603KRX7R9BB104" (at 294.64 156.21 0) (effects (font (size 1.524 1.524)) (hide yes)))
       (property "Description" "100nF local STM32 supply bypass; one per VDD/VDDA/USB supply group" (at 294.64 161.29 0) (effects (font (size 1.27 1.27)) (hide yes)))
       (pin "1")(pin "2")
@@
       (in_bom yes) (on_board yes) (dnp no)
  (property "Reference" "C37" (at 105.41 229.87 0) (effects (font (size 1.524 1.524)))) (property "Value" "100n" (at 105.41 233.68 0) (effects (font (size 1.524 1.524))))
-      (property "Footprint" "CountFidgetQ5:Capacitor_SMD_C_0603_1608Metric" (at 105.41 238.76 0) (effects (font (size 1.27 1.27)) (hide yes))) (property "MPN" "GRM188R71H104KA93D" (at 105.41 233.68 0) (effects (font (size 1.524 1.524)) (hide yes)))
+      (property "Footprint" "CountFidgetQ5:Capacitor_SMD_C_0603_1608Metric" (at 105.41 238.76 0) (effects (font (size 1.27 1.27)) (hide yes))) (property "MPN" "CC0603KRX7R9BB104" (at 105.41 233.68 0) (effects (font (size 1.524 1.524)) (hide yes)))
       (property "Description" "100nF charge reservoir for the 75k-source ADC input" (at 105.41 238.76 0) (effects (font (size 1.27 1.27)) (hide yes)))
       (pin "1")(pin "2")

Commit message: Move nine part types to JLC Basic; 16 Extended types remain, each justified
R4 18k (16.7 mA charge), temperature window 56k/82k/18k/12k (7.26-35.83 C),
R32 75 ohm, Q1/Q2 AO3400A, 2.2 uF and 10 uF 50 V 0805 capacitors. Fresh
ERC/DRC/parity on unchanged routing, stock 42/42, exports, JLC footprint
fit and pin names, power/latch checks re-run. About $28 less per order.

Co-Authored-By: Claude Opus 5.5 <noreply@anthropic.com>
Claude-Session: https://claude.ai/code/session_01UrkzLMrBi6iLPSL5SbMCA7
Parts:
- C6: MPN GRM21BR61E106KA73L -> GRM21BR61H106KE43L
Changed lines of the file:
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@@
       (in_bom yes) (on_board yes) (dnp no)
  (property "Reference" "C6" (at 294.64 229.87 0) (effects (font (size 1.524 1.524)))) (property "Value" "10u" (at 294.64 233.68 0) (effects (font (size 1.524 1.524))))
-      (property "Footprint" "CountFidgetQ5:Capacitor_SMD_C_0805_2012Metric" (at 294.64 238.76 0) (effects (font (size 1.27 1.27)) (hide yes))) (property "MPN" "GRM21BR61E106KA73L" (at 294.64 233.68 0) (effects (font (size 1.524 1.524)) (hide yes)))
-      (property "Description" "10uF package rail bulk; include all MCU/FRAM/module capacitance in regulator stability and startup review; effective capacitance unmeasured" (at 294.64 238.76 0) (effects (font (size 1.27 1.27)) (hide yes)))
+      (property "Footprint" "CountFidgetQ5:Capacitor_SMD_C_0805_2012Metric" (at 294.64 238.76 0) (effects (font (size 1.27 1.27)) (hide yes))) (property "MPN" "GRM21BR61H106KE43L" (at 294.64 233.68 0) (effects (font (size 1.524 1.524)) (hide yes)))
+      (property "Description" "10 uF, 50 V, X5R, 0805; effective >=1 uF at 4.5 V" (at 294.64 238.76 0) (effects (font (size 1.27 1.27)) (hide yes)))
       (pin "1")(pin "2")
       (instances (project "click-counter-Q5" (path "/7c190cd8-3ca2-5363-8a92-396d30a08243/25c8a497-d064-5849-8b98-8381803a397d" (reference "C6") (unit 1)))))
