File: electronics/q5/usb-power-1.kicad_sch (KiCad schematic)
At the start: 6 parts

Commit message: Q5 design lock: JLC Basic substitutions, re-verified board, cost estimator
Co-Authored-By: Claude Opus 5.5 <noreply@anthropic.com>
Claude-Session: https://claude.ai/code/session_01UrkzLMrBi6iLPSL5SbMCA7
Parts:
- C13, C29: MPN GRM1885C1H472JA01D -> 0603B472K500NT
- C38: MPN GRM188R71H104KA93D -> CC0603KRX7R9BB104
Changed lines of the file:
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@@
       (in_bom yes) (on_board yes) (dnp no)
  (property "Reference" "C13" (at 294.64 73.66 0) (effects (font (size 1.524 1.524)))) (property "Value" "4.7n" (at 294.64 77.46999999999998 0) (effects (font (size 1.524 1.524))))
-      (property "Footprint" "CountFidgetQ5:Capacitor_SMD_C_0603_1608Metric" (at 294.64 82.55 0) (effects (font (size 1.27 1.27)) (hide yes))) (property "MPN" "GRM1885C1H472JA01D" (at 294.64 77.46999999999998 0) (effects (font (size 1.524 1.524)) (hide yes)))
-      (property "Description" "4.7 nF, 50 V, C0G, 5%; same nominal TI EVM compensation ISET -> 2k -> 4.7n -> GND; low-current stability still requires measurement" (at 294.64 82.55 0) (effects (font (size 1.27 1.27)) (hide yes)))
+      (property "Footprint" "CountFidgetQ5:Capacitor_SMD_C_0603_1608Metric" (at 294.64 82.55 0) (effects (font (size 1.27 1.27)) (hide yes))) (property "MPN" "0603B472K500NT" (at 294.64 77.46999999999998 0) (effects (font (size 1.524 1.524)) (hide yes)))
+      (property "Description" "4.7 nF, 50 V, X7R, 5%; same nominal TI EVM compensation ISET -> 2k -> 4.7n -> GND; low-current stability still requires measurement" (at 294.64 82.55 0) (effects (font (size 1.27 1.27)) (hide yes)))
       (pin "1")(pin "2")
       (instances (project "click-counter-Q5" (path "/7c190cd8-3ca2-5363-8a92-396d30a08243/81d32175-1402-5eb1-8389-0a5fb2a4f6de" (reference "C13") (unit 1)))))
@@
       (in_bom yes) (on_board yes) (dnp no)
  (property "Reference" "C29" (at 294.64 152.4 0) (effects (font (size 1.524 1.524)))) (property "Value" "4.7n" (at 294.64 156.21 0) (effects (font (size 1.524 1.524))))
-      (property "Footprint" "CountFidgetQ5:Capacitor_SMD_C_0603_1608Metric" (at 294.64 161.29 0) (effects (font (size 1.27 1.27)) (hide yes))) (property "MPN" "GRM1885C1H472JA01D" (at 294.64 156.21 0) (effects (font (size 1.524 1.524)) (hide yes)))
-      (property "Description" "4.7nF 50V C0G slew capacitor to VIN; tON 17.9ms typical; typical slew only" (at 294.64 161.29 0) (effects (font (size 1.27 1.27)) (hide yes)))
+      (property "Footprint" "CountFidgetQ5:Capacitor_SMD_C_0603_1608Metric" (at 294.64 161.29 0) (effects (font (size 1.27 1.27)) (hide yes))) (property "MPN" "0603B472K500NT" (at 294.64 156.21 0) (effects (font (size 1.524 1.524)) (hide yes)))
+      (property "Description" "4.7nF 50V X7R slew capacitor to VIN; tON 17.9ms typical; typical slew only" (at 294.64 161.29 0) (effects (font (size 1.27 1.27)) (hide yes)))
       (pin "1")(pin "2")
       (instances (project "click-counter-Q5" (path "/7c190cd8-3ca2-5363-8a92-396d30a08243/81d32175-1402-5eb1-8389-0a5fb2a4f6de" (reference "C29") (unit 1)))))
@@
       (in_bom yes) (on_board yes) (dnp no)
  (property "Reference" "C38" (at 294.64 229.87 0) (effects (font (size 1.524 1.524)))) (property "Value" "100n" (at 294.64 233.68 0) (effects (font (size 1.524 1.524))))
-      (property "Footprint" "CountFidgetQ5:Capacitor_SMD_C_0603_1608Metric" (at 294.64 238.76 0) (effects (font (size 1.27 1.27)) (hide yes))) (property "MPN" "GRM188R71H104KA93D" (at 294.64 233.68 0) (effects (font (size 1.524 1.524)) (hide yes)))
+      (property "Footprint" "CountFidgetQ5:Capacitor_SMD_C_0603_1608Metric" (at 294.64 238.76 0) (effects (font (size 1.27 1.27)) (hide yes))) (property "MPN" "CC0603KRX7R9BB104" (at 294.64 233.68 0) (effects (font (size 1.524 1.524)) (hide yes)))
       (property "Description" "100nF local USBLC6 clamp-rail bypass, adjacent to D1/D2" (at 294.64 238.76 0) (effects (font (size 1.27 1.27)) (hide yes)))
       (pin "1")(pin "2")

Commit message: Move nine part types to JLC Basic; 16 Extended types remain, each justified
R4 18k (16.7 mA charge), temperature window 56k/82k/18k/12k (7.26-35.83 C),
R32 75 ohm, Q1/Q2 AO3400A, 2.2 uF and 10 uF 50 V 0805 capacitors. Fresh
ERC/DRC/parity on unchanged routing, stock 42/42, exports, JLC footprint
fit and pin names, power/latch checks re-run. About $28 less per order.

Co-Authored-By: Claude Opus 5.5 <noreply@anthropic.com>
Claude-Session: https://claude.ai/code/session_01UrkzLMrBi6iLPSL5SbMCA7
Parts:
- C1, C3: MPN GRM21BR71E225KE11L -> CL21A225KBQNNNE
- C2: MPN GRM21BR61E106KA73L -> GRM21BR61H106KE43L
Changed lines of the file:
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@@
       (in_bom yes) (on_board yes) (dnp no)
  (property "Reference" "C1" (at 105.41 73.66 0) (effects (font (size 1.524 1.524)))) (property "Value" "2.2u" (at 105.41 77.46999999999998 0) (effects (font (size 1.524 1.524))))
-      (property "Footprint" "CountFidgetQ5:Capacitor_SMD_C_0805_2012Metric" (at 105.41 82.55 0) (effects (font (size 1.27 1.27)) (hide yes))) (property "MPN" "GRM21BR71E225KE11L" (at 105.41 77.46999999999998 0) (effects (font (size 1.524 1.524)) (hide yes)))
-      (property "Description" "2.2 uF, 25 V, X7R; effective >=1 uF at 5 V" (at 105.41 82.55 0) (effects (font (size 1.27 1.27)) (hide yes)))
+      (property "Footprint" "CountFidgetQ5:Capacitor_SMD_C_0805_2012Metric" (at 105.41 82.55 0) (effects (font (size 1.27 1.27)) (hide yes))) (property "MPN" "CL21A225KBQNNNE" (at 105.41 77.46999999999998 0) (effects (font (size 1.524 1.524)) (hide yes)))
+      (property "Description" "2.2 uF, 50 V, X5R, 0805; effective >=1 uF at 5 V" (at 105.41 82.55 0) (effects (font (size 1.27 1.27)) (hide yes)))
       (pin "1")(pin "2")
       (instances (project "click-counter-Q5" (path "/7c190cd8-3ca2-5363-8a92-396d30a08243/81d32175-1402-5eb1-8389-0a5fb2a4f6de" (reference "C1") (unit 1)))))
@@
       (in_bom yes) (on_board yes) (dnp no)
  (property "Reference" "C2" (at 105.41 152.4 0) (effects (font (size 1.524 1.524)))) (property "Value" "10u" (at 105.41 156.21 0) (effects (font (size 1.524 1.524))))
-      (property "Footprint" "CountFidgetQ5:Capacitor_SMD_C_0805_2012Metric" (at 105.41 161.29 0) (effects (font (size 1.27 1.27)) (hide yes))) (property "MPN" "GRM21BR61E106KA73L" (at 105.41 156.21 0) (effects (font (size 1.524 1.524)) (hide yes)))
-      (property "Description" "10 uF, 25 V, X5R; effective >=1 uF at 4.5 V" (at 105.41 161.29 0) (effects (font (size 1.27 1.27)) (hide yes)))
+      (property "Footprint" "CountFidgetQ5:Capacitor_SMD_C_0805_2012Metric" (at 105.41 161.29 0) (effects (font (size 1.27 1.27)) (hide yes))) (property "MPN" "GRM21BR61H106KE43L" (at 105.41 156.21 0) (effects (font (size 1.524 1.524)) (hide yes)))
+      (property "Description" "10 uF, 50 V, X5R, 0805; effective >=1 uF at 4.5 V" (at 105.41 161.29 0) (effects (font (size 1.27 1.27)) (hide yes)))
       (pin "1")(pin "2")
       (instances (project "click-counter-Q5" (path "/7c190cd8-3ca2-5363-8a92-396d30a08243/81d32175-1402-5eb1-8389-0a5fb2a4f6de" (reference "C2") (unit 1)))))
@@
       (in_bom yes) (on_board yes) (dnp no)
  (property "Reference" "C3" (at 105.41 229.87 0) (effects (font (size 1.524 1.524)))) (property "Value" "2.2u" (at 105.41 233.68 0) (effects (font (size 1.524 1.524))))
-      (property "Footprint" "CountFidgetQ5:Capacitor_SMD_C_0805_2012Metric" (at 105.41 238.76 0) (effects (font (size 1.27 1.27)) (hide yes))) (property "MPN" "GRM21BR71E225KE11L" (at 105.41 233.68 0) (effects (font (size 1.524 1.524)) (hide yes)))
-      (property "Description" "2.2 uF, 25 V, X7R" (at 105.41 238.76 0) (effects (font (size 1.27 1.27)) (hide yes)))
+      (property "Footprint" "CountFidgetQ5:Capacitor_SMD_C_0805_2012Metric" (at 105.41 238.76 0) (effects (font (size 1.27 1.27)) (hide yes))) (property "MPN" "CL21A225KBQNNNE" (at 105.41 233.68 0) (effects (font (size 1.524 1.524)) (hide yes)))
+      (property "Description" "2.2 uF, 50 V, X5R, 0805; effective >=1 uF at 5 V" (at 105.41 238.76 0) (effects (font (size 1.27 1.27)) (hide yes)))
       (pin "1")(pin "2")
       (instances (project "click-counter-Q5" (path "/7c190cd8-3ca2-5363-8a92-396d30a08243/81d32175-1402-5eb1-8389-0a5fb2a4f6de" (reference "C3") (unit 1)))))
