File: electronics/q5/usb-power-2.kicad_sch (KiCad schematic)
At the start: 6 parts

Commit message: WIP: Q5 design-lock routing iteration snapshot (not verified)
Co-Authored-By: Claude Opus 5.5 <noreply@anthropic.com>
Claude-Session: https://claude.ai/code/session_01UrkzLMrBi6iLPSL5SbMCA7
Parts:
- removed D4: 1N4148WS, CountFidgetQ5:Diode_SMD_D_SOD-323, symbol CountFidgetQ5:D4
- added C40: 4.7n, CountFidgetQ5:Capacitor_SMD_C_0603_1608Metric, symbol CountFidgetQ5:C40
Connections:
- net GND: now also C40.2
- net SYS_ON: now also C40.1
Other:
- moved on the sheet: C5, D1, D2, D3

Commit message: Q5 design lock: JLC Basic substitutions, re-verified board, cost estimator
Co-Authored-By: Claude Opus 5.5 <noreply@anthropic.com>
Claude-Session: https://claude.ai/code/session_01UrkzLMrBi6iLPSL5SbMCA7
Parts:
- C39: MPN GRM188R71H104KA93D -> CC0603KRX7R9BB104
- C40: MPN GRM1885C1H472JA01D -> 0603B472K500NT
Changed lines of the file:
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@@
       (in_bom yes) (on_board yes) (dnp no)
  (property "Reference" "C39" (at 105.41 73.66 0) (effects (font (size 1.524 1.524)))) (property "Value" "100n" (at 105.41 77.46999999999998 0) (effects (font (size 1.524 1.524))))
-      (property "Footprint" "CountFidgetQ5:Capacitor_SMD_C_0603_1608Metric" (at 105.41 82.55 0) (effects (font (size 1.27 1.27)) (hide yes))) (property "MPN" "GRM188R71H104KA93D" (at 105.41 77.46999999999998 0) (effects (font (size 1.524 1.524)) (hide yes)))
+      (property "Footprint" "CountFidgetQ5:Capacitor_SMD_C_0603_1608Metric" (at 105.41 82.55 0) (effects (font (size 1.27 1.27)) (hide yes))) (property "MPN" "CC0603KRX7R9BB104" (at 105.41 77.46999999999998 0) (effects (font (size 1.524 1.524)) (hide yes)))
       (property "Description" "100nF local USBLC6 clamp-rail bypass, adjacent to D1/D2" (at 105.41 82.55 0) (effects (font (size 1.27 1.27)) (hide yes)))
       (pin "1")(pin "2")
@@
       (in_bom yes) (on_board yes) (dnp no)
  (property "Reference" "C40" (at 294.64 73.66 0) (effects (font (size 1.524 1.524)))) (property "Value" "4.7n" (at 294.64 77.46999999999998 0) (effects (font (size 1.524 1.524))))
-      (property "Footprint" "CountFidgetQ5:Capacitor_SMD_C_0603_1608Metric" (at 294.64 82.55 0) (effects (font (size 1.27 1.27)) (hide yes))) (property "MPN" "GRM1885C1H472JA01D" (at 294.64 77.46999999999998 0) (effects (font (size 1.524 1.524)) (hide yes)))
-      (property "Description" "4.7nF C0G on U7 ON: holds ON through COUNT-key contact bounce (tau with R35 = 4.7 ms); U7 turns off ~10 ms after the last source is released." (at 294.64 82.55 0) (effects (font (size 1.27 1.27)) (hide yes)))
+      (property "Footprint" "CountFidgetQ5:Capacitor_SMD_C_0603_1608Metric" (at 294.64 82.55 0) (effects (font (size 1.27 1.27)) (hide yes))) (property "MPN" "0603B472K500NT" (at 294.64 77.46999999999998 0) (effects (font (size 1.524 1.524)) (hide yes)))
+      (property "Description" "4.7nF X7R on U7 ON: holds ON through COUNT-key contact bounce (tau with R35 = 4.7 ms); U7 turns off ~10 ms after the last source is released." (at 294.64 82.55 0) (effects (font (size 1.27 1.27)) (hide yes)))
       (pin "1")(pin "2")
       (instances (project "click-counter-Q5" (path "/7c190cd8-3ca2-5363-8a92-396d30a08243/212a85d9-b47b-5df6-8d9b-ffcc17a81200" (reference "C40") (unit 1)))))

Commit message: First-order de-risking: U5 supply filter, 10 nF latch cap, JLC-corrected CPLs, DFU unplug rule
Three independent checks (datasheet pinouts, JLC EasyEDA footprints, dead-on-arrival
review) found no pinout, footprint or DOA defect. Changes from their findings:
R39 1k + C9 filter U5's 6 V abs-max supply from VBUS hot-plug ringing; C40 10 nF
(min latch press 10.5 ms typ); JLC-corrected CPL files and a preview checklist;
flasher warns to reset a unit left in DFU before unplugging. Board re-routed:
DRC/ERC/parity zero, no via-to-land gaps; emulator 0 failures; stock 43/43.

Co-Authored-By: Claude Opus 5.5 <noreply@anthropic.com>
Claude-Session: https://claude.ai/code/session_01UrkzLMrBi6iLPSL5SbMCA7
Parts:
- C40: value 4.7n -> 10n; MPN 0603B472K500NT -> 0603B103K500NT
Changed lines of the file:
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@@
 (symbol (lib_id "CountFidgetQ5:C40") (at 294.64 82.55 0) (unit 1) (exclude_from_sim no)
       (in_bom yes) (on_board yes) (dnp no)
- (property "Reference" "C40" (at 294.64 73.66 0) (effects (font (size 1.524 1.524)))) (property "Value" "4.7n" (at 294.64 77.46999999999998 0) (effects (font (size 1.524 1.524))))
-      (property "Footprint" "CountFidgetQ5:Capacitor_SMD_C_0603_1608Metric" (at 294.64 82.55 0) (effects (font (size 1.27 1.27)) (hide yes))) (property "MPN" "0603B472K500NT" (at 294.64 77.46999999999998 0) (effects (font (size 1.524 1.524)) (hide yes)))
-      (property "Description" "4.7nF X7R on U7 ON: holds ON through COUNT-key contact bounce (tau with R35 = 4.7 ms); U7 turns off ~10 ms after the last source is released." (at 294.64 82.55 0) (effects (font (size 1.27 1.27)) (hide yes)))
+ (property "Reference" "C40" (at 294.64 73.66 0) (effects (font (size 1.524 1.524)))) (property "Value" "10n" (at 294.64 77.46999999999998 0) (effects (font (size 1.524 1.524))))
+      (property "Footprint" "CountFidgetQ5:Capacitor_SMD_C_0603_1608Metric" (at 294.64 82.55 0) (effects (font (size 1.27 1.27)) (hide yes))) (property "MPN" "0603B103K500NT" (at 294.64 77.46999999999998 0) (effects (font (size 1.524 1.524)) (hide yes)))
+      (property "Description" "10nF X7R on U7 ON: holds ON through COUNT-key contact bounce (tau with R35 = 10 ms); U7 turns off ~21 ms after the last source is released." (at 294.64 82.55 0) (effects (font (size 1.27 1.27)) (hide yes)))
       (pin "1")(pin "2")
       (instances (project "click-counter-Q5" (path "/7c190cd8-3ca2-5363-8a92-396d30a08243/212a85d9-b47b-5df6-8d9b-ffcc17a81200" (reference "C40") (unit 1)))))

Commit message: Move nine part types to JLC Basic; 16 Extended types remain, each justified
R4 18k (16.7 mA charge), temperature window 56k/82k/18k/12k (7.26-35.83 C),
R32 75 ohm, Q1/Q2 AO3400A, 2.2 uF and 10 uF 50 V 0805 capacitors. Fresh
ERC/DRC/parity on unchanged routing, stock 42/42, exports, JLC footprint
fit and pin names, power/latch checks re-run. About $28 less per order.

Co-Authored-By: Claude Opus 5.5 <noreply@anthropic.com>
Claude-Session: https://claude.ai/code/session_01UrkzLMrBi6iLPSL5SbMCA7
Parts:
- C5: MPN GRM21BR71E225KE11L -> CL21A225KBQNNNE
Changed lines of the file:
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@@
       (in_bom yes) (on_board yes) (dnp no)
  (property "Reference" "C5" (at 105.41 152.4 0) (effects (font (size 1.524 1.524)))) (property "Value" "2.2u" (at 105.41 156.21 0) (effects (font (size 1.524 1.524))))
-      (property "Footprint" "CountFidgetQ5:Capacitor_SMD_C_0805_2012Metric" (at 105.41 161.29 0) (effects (font (size 1.27 1.27)) (hide yes))) (property "MPN" "GRM21BR71E225KE11L" (at 105.41 156.21 0) (effects (font (size 1.524 1.524)) (hide yes)))
-      (property "Description" "" (at 105.41 161.29 0) (effects (font (size 1.27 1.27)) (hide yes)))
+      (property "Footprint" "CountFidgetQ5:Capacitor_SMD_C_0805_2012Metric" (at 105.41 161.29 0) (effects (font (size 1.27 1.27)) (hide yes))) (property "MPN" "CL21A225KBQNNNE" (at 105.41 156.21 0) (effects (font (size 1.524 1.524)) (hide yes)))
+      (property "Description" "2.2 uF, 50 V, X5R, 0805; effective >=1 uF at 5 V" (at 105.41 161.29 0) (effects (font (size 1.27 1.27)) (hide yes)))
       (pin "1")(pin "2")
       (instances (project "click-counter-Q5" (path "/7c190cd8-3ca2-5363-8a92-396d30a08243/212a85d9-b47b-5df6-8d9b-ffcc17a81200" (reference "C5") (unit 1)))))
